File: Interface_Board/Sirius_Interface_Board.kicad_pcb (KiCad board)
At the start: 2 copper layers, 157 x 65 mm, 20 parts, among them J1 KB1, J10 TO_VIDEO, J11 JOYSTICK, J12 TO_JOYSTICK, J13 TO_RESET, J15 DIN5, J2 TO_KB1, J3 KB2, J4 TO_KB2, J5 POWER, J6 TO_POWER, J7 TAPE, J8 TO_TAPE, J9 AUDIO, SW1 RESET

Commit message: Minor changes to interface board
Parts:
- moved H6 64.4 mm to (170.2, 111.2)
- moved H1 64.4 mm to (56.2, 70.2)
- moved H3 64.4 mm to (206.2, 70.2)
- moved H4 64.4 mm to (56.2, 93.2)
- moved J10 64.4 mm to (107.8, 86.5)
- moved J12 64.4 mm to (190.5, 86.2)
- moved J15 64.4 mm to (112.9, 78.6)
- moved J5 64.4 mm to (70.1, 82.0)
- moved H5 64.4 mm to (206.2, 128.2)
- moved J1 64.4 mm to (165.7, 128.6)
- moved J11 64.4 mm to (190.5, 77.6)
- moved J13 64.4 mm to (150.8, 89.6)
- moved J2 64.4 mm to (163.5, 110.8)
- moved J3 64.4 mm to (63.2, 90.6)
- moved J4 64.4 mm to (180.9, 128.6)
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Routing:
- net +5V: track 137.7 -> 134.3 mm
Other:
- board text added: "AUDIO"
- board text added: "Oct 2025"
- board text removed: "June 2025"
