File: Interface_Board/Sirius_Interface_Board.kicad_sch (KiCad schematic)
At the start: 20 parts, among them J1 KB1, J10 TO_VIDEO, J11 JOYSTICK, J12 TO_JOYSTICK, J13 TO_RESET, J15 DIN5, J2 TO_KB1, J3 KB2, J4 TO_KB2, J5 POWER, J6 TO_POWER, J7 TAPE, J8 TO_TAPE, J9 AUDIO, SW1 RESET

Commit message: Minor changes to interface board
Other:
- company: (none) -> www.youtube.com/@Brfff
- title: (none) -> Interface Board for Сириус
Changed lines of the file:
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@@
 	(generator_version "9.0")
 	(paper "A4")
+	(title_block
+		(title "Interface Board for Сириус")
+		(date "31/OCT/2025")
+		(rev "B")
+		(company "www.youtube.com/@Brfff")
+	)
 	(text_box "Atari Joystick\nPin 1 = UP\nPin 2 = DOWN\nPin 3 = LEFT\nPin 4 = RIGHT\nPin 5 = n/c\nPin 6 = FIRE\nPin 7 = +5V\nPin 8 = GND\nPin 9 = n/c"
 		(exclude_from_sim no)
